File: 20kz_midi2cv.sch (KiCad schematic (older format))
At the start: 17 parts

Commit message: a falta de ajustar la tensión de salida para que cubra un rango de 8 octavas, es decir 8 voltios
Parts:
- C? (x2): value C -> 22p
- C?: value 10u -> 0.33u
- C?: value 10u -> 0.1u
- U?: symbol 4N25 -> 4N25-RESCUE-20kz_midi2cv
Connections:
- net labels added: +5V, +9V
- net labels removed: VCC, vcc
- wire segments 41 -> 85
Other:
- note added: "DAC\n"
- note added: "MIDI out"
- note added: "Microcontroller"
- note added: "Power\n"
- moved on the sheet: C?, D?, J?, R?, U?, Y?

Commit message: ...
Parts:
- removed C?: 0.33u, symbol CP
- removed C?: 0.1u, symbol CP
- removed D?: LED, symbol LED
- removed J?: BARREL_JACK, symbol BARREL_JACK
- removed R?: 220, symbol R
- removed U?: 7805, symbol 7805
- added J?: TONE, symbol Audio-Jack-2
- added J?: PITCH BEND, symbol Audio-Jack-2
- added J? (x2): GATE, symbol Audio-Jack-2
- added Q? (x2): 2N3904, TO_SOT_Packages_THT:TO-92_Molded_Narrow, symbol 2N3904
- added R? (x2): 5K, symbol R
- added R? (x2): 1K, symbol R
- added RV? (x2): POT, symbol POT
- added U? (x2): LM358, symbol LM358
Connections:
- net +5V: now also Q?.3 (C), Q?.3 (C)
- net GND: now also J?.2, J?.2, J?.2, J?.2, R?.1, R?.1, RV?.2, RV?.2, RV?.3, RV?.3
- net GATE: now reaches U?.4 ((PCINT18/INT0)PD2)
- net GATE: now also Q?.2 (B)
- net TRIG: now reaches U?.6 ((PCINT20/XCK/T0)PD4)
- net TRIG: now also Q?.2 (B)
- net DAC-B: now reaches U?.10 (VoutB)
- net DAC-B: now also U?.3 (+)
- net DAC-A: now reaches U?.14 (VoutA)
- net DAC-A: now also U?.3 (+)
- new net: J?.1, R?.1, U?.1 (x2)
- new net: R?.2, RV?.1, U?.2 (-) (x2)
- new net: J?.1, Q?.1 (E), R?.2 (x2)
- new net +15V: U?.8 (V+), U?.8 (V+)
- new net -15V: U?.4 (V-), U?.4 (V-)
Other:
- note added: "Gate control"
- note added: "MIDI receiver"
- note added: "Pitch bend control"
- note added: "Tone control"
- note added: "Trigger control"
- note added: "calibration"
- note removed: "MIDI out"
- note removed: "Power\n"
- moved on the sheet: C?, D?, J?, R?, U?, Y?

Commit message: reglas crc ok
Parts:
- added J6: power, symbol Conn_01x04
- gave numbers to parts that had none: 24
Connections:
- net +15V: now also J6.2 (Pin_2)
- net +5V: now also J6.1 (Pin_1); no longer U2.21 (AREF)
- net -15V: now also J6.3 (Pin_3)
- net DAC-B: now also U4.5 (+); no longer U4.3 (+)
- net GND: now also J6.4 (Pin_4)
- net at J5.1, R7.1: now also U4.7; no longer U4.1
- net at R7.2, RV2.1: now also U4.6 (-); no longer U4.2 (-)
- no-connect marks 0 -> 18
Other:
- moved on the sheet: D1, J1, R1, R2, U1

Commit message: añado condensadores a la entrada de 5V del micro y del DAC
Parts:
- added C3, C4: 100n, symbol C
Connections:
- net +5V: now also C3.1, C4.2
- net GND: now also C3.2, C4.1
Changed lines of the file:
@@
 $EndComp
 $Comp
-L GND #PWR01
+L GND #PWR13
 U 1 1 59BFD3CC
 P 3450 2800
-F 0 "#PWR01" H 3450 2550 50  0001 C CNN
+F 0 "#PWR13" H 3450 2550 50  0001 C CNN
 F 1 "GND" H 3450 2650 50  0000 C CNN
 F 2 "" H 3450 2800 50  0001 C CNN
@@
 $EndComp
 $Comp
-L GND #PWR02
+L GND #PWR16
 U 1 1 59BFDB2E
 P 5000 3550
-F 0 "#PWR02" H 5000 3300 50  0001 C CNN
+F 0 "#PWR16" H 5000 3300 50  0001 C CNN
 F 1 "GND" H 5000 3400 50  0000 C CNN
 F 2 "" H 5000 3550 50  0001 C CNN
@@
 $EndComp
 $Comp
-L GND #PWR03
+L GND #PWR9
 U 1 1 59BFF0AF
 P 8300 2000
-F 0 "#PWR03" H 8300 1750 50  0001 C CNN
+F 0 "#PWR9" H 8300 1750 50  0001 C CNN
 F 1 "GND" H 8300 1850 50  0000 C CNN
 F 2 "" H 8300 2000 50  0001 C CNN
@@
 RX
 $Comp
-L GND #PWR04
+L GND #PWR14
 U 1 1 59C28A87
 P 9450 3050
-F 0 "#PWR04" H 9450 2800 50  0001 C CNN
+F 0 "#PWR14" H 9450 2800 50  0001 C CNN
 F 1 "GND" H 9450 2900 50  0000 C CNN
 F 2 "" H 9450 3050 50  0001 C CNN
@@
 Text Notes 2050 2050 0    60   ~ 0
 MIDI receiver
-Text Notes 9450 1500 0    60   ~ 0
+Text Notes 9550 1200 0    60   ~ 0
 DAC\n
 Text Notes 5750 850  0    60   ~ 0
 Microcontroller
 $Comp
-L +5V #PWR05
+L +5V #PWR10
 U 1 1 59C2B213
 P 3450 2050
-F 0 "#PWR05" H 3450 1900 50  0001 C CNN
+F 0 "#PWR10" H 3450 1900 50  0001 C CNN
 F 1 "+5V" H 3450 2190 50  0000 C CNN
 F 2 "" H 3450 2050 50  0001 C CNN
@@
 $EndComp
 $Comp
-L +5V #PWR06
+L +5V #PWR2
 U 1 1 59C2B4B2
 P 4950 1150
-F 0 "#PWR06" H 4950 1000 50  0001 C CNN
+F 0 "#PWR2" H 4950 1000 50  0001 C CNN
 F 1 "+5V" H 4950 1290 50  0000 C CNN
 F 2 "" H 4950 1150 50  0001 C CNN
@@
 $EndComp
 $Comp
-L +5V #PWR07
+L +5V #PWR7
 U 1 1 59C2B740
-P 9450 1800
-F 0 "#PWR07" H 9450 1650 50  0001 C CNN
-F 1 "+5V" H 9450 1940 50  0000 C CNN
-F 2 "" H 9450 1800 50  0001 C CNN
-F 3 "" H 9450 1800 50  0001 C CNN
-	1    9450 1800
-	1    0    0    -1
-$EndComp
-$Comp
-L +5V #PWR08
+P 9450 1500
+F 0 "#PWR7" H 9450 1350 50  0001 C CNN
+F 1 "+5V" H 9450 1640 50  0000 C CNN
+F 2 "" H 9450 1500 50  0001 C CNN
+F 3 "" H 9450 1500 50  0001 C CNN
+	1    9450 1500
+	1    0    0    -1
+$EndComp
+$Comp
+L +5V #PWR15
 U 1 1 59C2B949
 P 9650 3050
-F 0 "#PWR08" H 9650 2900 50  0001 C CNN
+F 0 "#PWR15" H 9650 2900 50  0001 C CNN
 F 1 "+5V" H 9650 3190 50  0000 C CNN
 F 2 "" H 9650 3050 50  0001 C CNN
@@
 $EndComp
 $Comp
-L +5V #PWR09
+L +5V #PWR11
 U 1 1 59C2BF25
 P 7700 2600
-F 0 "#PWR09" H 7700 2450 50  0001 C CNN
+F 0 "#PWR11" H 7700 2450 50  0001 C CNN
 F 1 "+5V" H 7700 2740 50  0000 C CNN
 F 2 "" H 7700 2600 50  0001 C CNN
@@
 $EndComp
 $Comp
-L +5V #PWR010
+L +5V #PWR12
 U 1 1 59C2C020
 P 8750 2650
-F 0 "#PWR010" H 8750 2500 50  0001 C CNN
+F 0 "#PWR12" H 8750 2500 50  0001 C CNN
 F 1 "+5V" H 8750 2790 50  0000 C CNN
 F 2 "" H 8750 2650 50  0001 C CNN
@@
 	9450 2950 9450 3050
 Wire Wire Line
-	9450 1800 9450 1950
+	9450 1500 9450 1950
 Wire Wire Line
 	7000 1150 7200 1150
@@
 	7000 1750 7200 1750
 Wire Wire Line
-	4950 1150 5100 1150
+	4800 1150 5100 1150
 Wire Wire Line
 	7500 2600 7700 2600
@@
 $EndComp
 $Comp
-L +15V #PWR011
+L +15V #PWR17
 U 1 1 59C3649C
 P 1800 3750
-F 0 "#PWR011" H 1800 3600 50  0001 C CNN
+F 0 "#PWR17" H 1800 3600 50  0001 C CNN
 F 1 "+15V" H 1800 3890 50  0000 C CNN
 F 2 "" H 1800 3750 50  0001 C CNN
@@
 $EndComp
 $Comp
-L -15V #PWR17
+L -15V #PWR19
 U 1 1 59C364C8
 P 1800 4350
-F 0 "#PWR17" H 1800 4450 50  0001 C CNN
+F 0 "#PWR19" H 1800 4450 50  0001 C CNN
 F 1 "-15V" H 1800 4500 50  0000 C CNN
 F 2 "" H 1800 4350 50  0001 C CNN
@@
 	10150 2250 10350 2250
 $Comp
-L GND #PWR012
+L GND #PWR22
 U 1 1 59C37211
 P 1450 5050
-F 0 "#PWR012" H 1450 4800 50  0001 C CNN
+F 0 "#PWR22" H 1450 4800 50  0001 C CNN
 F 1 "GND" H 1450 4900 50  0000 C CNN
 F 2 "" H 1450 5050 50  0001 C CNN
@@
 Connection ~ 2350 4050
 $Comp
-L GND #PWR013
+L GND #PWR18
 U 1 1 59C38A05
 P 2650 4300
-F 0 "#PWR013" H 2650 4050 50  0001 C CNN
+F 0 "#PWR18" H 2650 4050 50  0001 C CNN
 F 1 "GND" H 2650 4150 50  0000 C CNN
 F 2 "" H 2650 4300 50  0001 C CNN
@@
 $EndComp
 $Comp
-L +15V #PWR014
+L +15V #PWR23
 U 1 1 59C38F5B
 P 1800 5450
-F 0 "#PWR014" H 1800 5300 50  0001 C CNN
+F 0 "#PWR23" H 1800 5300 50  0001 C CNN
 F 1 "+15V" H 1800 5590 50  0000 C CNN
 F 2 "" H 1800 5450 50  0001 C CNN
@@
 $EndComp
 $Comp
-L -15V #PWR27
+L -15V #PWR29
 U 1 1 59C38F61
 P 1800 6050
-F 0 "#PWR27" H 1800 6150 50  0001 C CNN
+F 0 "#PWR29" H 1800 6150 50  0001 C CNN
 F 1 "-15V" H 1800 6200 50  0000 C CNN
 F 2 "" H 1800 6050 50  0001 C CNN
@@
 $EndComp
 $Comp
-L GND #PWR015
+L GND #PWR30
 U 1 1 59C38F75
 P 1450 6750
-F 0 "#PWR015" H 1450 6500 50  0001 C CNN
+F 0 "#PWR30" H 1450 6500 50  0001 C CNN
 F 1 "GND" H 1450 6600 50  0000 C CNN
 F 2 "" H 1450 6750 50  0001 C CNN
@@
 Connection ~ 2350 5750
 $Comp
-L GND #PWR016
+L GND #PWR28
 U 1 1 59C38F8F
 P 2650 6000
-F 0 "#PWR016" H 2650 5750 50  0001 C CNN
+F 0 "#PWR28" H 2650 5750 50  0001 C CNN
 F 1 "GND" H 2650 5850 50  0000 C CNN
 F 2 "" H 2650 6000 50  0001 C CNN
@@
 $EndComp
 $Comp
-L GND #PWR017
+L GND #PWR24
 U 1 1 59C39D84
 P 5850 5500
-F 0 "#PWR017" H 5850 5250 50  0001 C CNN
+F 0 "#PWR24" H 5850 5250 50  0001 C CNN
 F 1 "GND" H 5850 5350 50  0000 C CNN
 F 2 "" H 5850 5500 50  0001 C CNN
@@
 $EndComp
 $Comp
-L +5V #PWR018
+L +5V #PWR20
 U 1 1 59C3A03A
 P 5850 4550
-F 0 "#PWR018" H 5850 4400 50  0001 C CNN
+F 0 "#PWR20" H 5850 4400 50  0001 C CNN
 F 1 "+5V" H 5850 4690 50  0000 C CNN
 F 2 "" H 5850 4550 50  0001 C CNN
@@
 Connection ~ 5850 5100
 $Comp
-L GND #PWR019
+L GND #PWR25
 U 1 1 59C3A4C6
 P 6150 5500
-F 0 "#PWR019" H 6150 5250 50  0001 C CNN
+F 0 "#PWR25" H 6150 5250 50  0001 C CNN
 F 1 "GND" H 6150 5350 50  0000 C CNN
 F 2 "" H 6150 5500 50  0001 C CNN
@@
 $EndComp
 $Comp
-L GND #PWR020
+L GND #PWR26
 U 1 1 59C3A967
 P 8100 5500
-F 0 "#PWR020" H 8100 5250 50  0001 C CNN
+F 0 "#PWR26" H 8100 5250 50  0001 C CNN
 F 1 "GND" H 8100 5350 50  0000 C CNN
 F 2 "" H 8100 5500 50  0001 C CNN
@@
 $EndComp
 $Comp
-L +5V #PWR021
+L +5V #PWR21
 U 1 1 59C3A973
 P 8100 4550
-F 0 "#PWR021" H 8100 4400 50  0001 C CNN
+F 0 "#PWR21" H 8100 4400 50  0001 C CNN
 F 1 "+5V" H 8100 4690 50  0000 C CNN
 F 2 "" H 8100 4550 50  0001 C CNN
@@
 Connection ~ 8100 5100
 $Comp
-L GND #PWR022
+L GND #PWR27
 U 1 1 59C3A985
 P 8400 5500
-F 0 "#PWR022" H 8400 5250 50  0001 C CNN
+F 0 "#PWR27" H 8400 5250 50  0001 C CNN
 F 1 "GND" H 8400 5350 50  0000 C CNN
 F 2 "" H 8400 5500 50  0001 C CNN
@@
 $EndComp
 $Comp
-L +5V #PWR023
+L +5V #PWR1
 U 1 1 59C3CE9F
 P 2100 1150
-F 0 "#PWR023" H 2100 1000 50  0001 C CNN
+F 0 "#PWR1" H 2100 1000 50  0001 C CNN
 F 1 "+5V" H 2100 1290 50  0000 C CNN
 F 2 "" H 2100 1150 50  0001 C CNN
@@
 $EndComp
 $Comp
-L +15V #PWR024
+L +15V #PWR3
 U 1 1 59C3CF60
 P 2400 1250
-F 0 "#PWR024" H 2400 1100 50  0001 C CNN
+F 0 "#PWR3" H 2400 1100 50  0001 C CNN
 F 1 "+15V" H 2400 1390 50  0000 C CNN
 F 2 "" H 2400 1250 50  0001 C CNN
@@
 $EndComp
 $Comp
-L GND #PWR025
+L GND #PWR5
 U 1 1 59C3D43E
 P 2100 1450
-F 0 "#PWR025" H 2100 1200 50  0001 C CNN
+F 0 "#PWR5" H 2100 1200 50  0001 C CNN
 F 1 "GND" H 2100 1300 50  0000 C CNN
 F 2 "" H 2100 1450 50  0001 C CNN
@@
 	1900 1450 2100 1450
 $Comp
-L PWR_FLAG #FLG026
+L PWR_FLAG #FLG1
 U 1 1 59C3DC74
 P 2100 1150
-F 0 "#FLG026" H 2100 1225 50  0001 C CNN
+F 0 "#FLG1" H 2100 1225 50  0001 C CNN
 F 1 "PWR_FLAG" H 2100 1300 50  0001 C CNN
 F 2 "" H 2100 1150 50  0001 C CNN
@@
 $EndComp
 $Comp
-L PWR_FLAG #FLG027
+L PWR_FLAG #FLG2
 U 1 1 59C3DD8A
 P 2400 1250
-F 0 "#FLG027" H 2400 1325 50  0001 C CNN
+F 0 "#FLG2" H 2400 1325 50  0001 C CNN
 F 1 "PWR_FLAG" H 2400 1400 50  0001 C CNN
 F 2 "" H 2400 1250 50  0001 C CNN
@@
 $EndComp
 $Comp
-L PWR_FLAG #FLG028
+L PWR_FLAG #FLG3
 U 1 1 59C3DDE3
 P 2700 1350
-F 0 "#FLG028" H 2700 1425 50  0001 C CNN
+F 0 "#FLG3" H 2700 1425 50  0001 C CNN
 F 1 "PWR_FLAG" H 2700 1500 50  0001 C CNN
 F 2 "" H 2700 1350 50  0001 C CNN
@@
 $EndComp
 $Comp
-L PWR_FLAG #FLG029
+L PWR_FLAG #FLG4
 U 1 1 59C3DFB5
 P 2100 1450
-F 0 "#FLG029" H 2100 1525 50  0001 C CNN
+F 0 "#FLG4" H 2100 1525 50  0001 C CNN
 F 1 "PWR_FLAG" H 2100 1600 50  0001 C CNN
 F 2 "" H 2100 1450 50  0001 C CNN
@@
 NoConn ~ 1800 2700
 NoConn ~ 5100 1750
+$Comp
+L C C3
+U 1 1 59C4EC2E
+P 4800 1300
+F 0 "C3" H 4825 1400 50  0000 L CNN
+F 1 "100n" H 4825 1200 50  0000 L CNN
+F 2 "" H 4838 1150 50  0001 C CNN
+F 3 "" H 4800 1300 50  0001 C CNN
+	1    4800 1300
+	1    0    0    -1
+$EndComp
+$Comp
+L GND #PWR6
+U 1 1 59C4ECB6
+P 4800 1500
+F 0 "#PWR6" H 4800 1250 50  0001 C CNN
+F 1 "GND" H 4800 1350 50  0000 C CNN
+F 2 "" H 4800 1500 50  0001 C CNN
+F 3 "" H 4800 1500 50  0001 C CNN
+	1    4800 1500
+	1    0    0    -1
+$EndComp
+Wire Wire Line
+	4800 1450 4800 1500
+Connection ~ 4950 1150
+$Comp
+L C C4
+U 1 1 59C4F198
+P 9700 1600
+F 0 "C4" H 9725 1700 50  0000 L CNN
+F 1 "100n" H 9725 1500 50  0000 L CNN
+F 2 "" H 9738 1450 50  0001 C CNN
+F 3 "" H 9700 1600 50  0001 C CNN
+	1    9700 1600
+	0    1    1    0
+$EndComp
+$Comp
+L GND #PWR8
+U 1 1 59C4F19E
+P 9950 1650
+F 0 "#PWR8" H 9950 1400 50  0001 C CNN
+F 1 "GND" H 9950 1500 50  0000 C CNN
+F 2 "" H 9950 1650 50  0001 C CNN
+F 3 "" H 9950 1650 50  0001 C CNN
+	1    9950 1650
+	1    0    0    -1
+$EndComp
+Wire Wire Line
+	9850 1600 9950 1600
+Wire Wire Line
+	9950 1600 9950 1650
+Wire Wire Line
+	9550 1600 9450 1600
+Connection ~ 9450 1600
 $EndSCHEMATC
